File: corne-light.kicad_pcb (KiCad board)
At the start: 2 copper layers, 273 x 91.4 mm, 117 parts, among them J2 OLED, J3 Conn_01x02, J4 Conn_01x02, J6 AudioJack4, J7 OLED, J8 AudioJack4, SW1 SW_PUSH, SW10 SW_PUSH, SW11 SW_PUSH, SW12 SW_PUSH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

Commit message: update prod files and project to v9
Parts:
- moved J8 0.20 mm to (20.9, 105.7)
- moved J6 0.20 mm to (286.5, 110.3)
