File: corne-light.kicad_sch (KiCad schematic)
At the start: 96 parts, among them J1 MJ-4PP-9, J2 OLED, J3 Conn_01x02, J4 Conn_01x02, J6 MJ-4PP-9, J7 OLED, SW1 SW_PUSH, SW10 SW_PUSH, SW11 SW_PUSH, SW12 SW_PUSH, SW13 SW_PUSH, SW14 SW_PUSH, SW15 SW_PUSH, SW16 SW_PUSH, SW17 SW_PUSH, SW18 SW_PUSH, SW19 SW_PUSH, SW2 SW_PUSH, SW20 SW_PUSH, SW21 SW_PUSH, SW22 SW_PUSH, SW23 SW_PUSH, SW24 SW_PUSH, SW25 SW_PUSH, SW26 SW_PUSH, SW27 SW_PUSH, SW28 SW_PUSH, SW29 SW_PUSH, SW3 SW_PUSH, SW30 SW_PUSH, SW31 SW_PUSH, SW32 SW_PUSH, SW33 SW_PUSH, SW34 SW_PUSH, SW35 SW_PUSH, SW36 SW_PUSH, SW37 SW_PUSH, SW38 SW_PUSH, SW39 SW_PUSH, SW4 SW_PUSH, SW40 SW_PUSH, SW41 SW_PUSH, SW42 SW_PUSH, SW44 SW_Slide_DPDT, SW45 SW_Slide_DPDT, SW5 SW_PUSH, SW6 SW_PUSH, SW7 SW_PUSH, SW8 SW_PUSH, SW9 SW_PUSH, U1 nice_nano, U2 nice_nano

Commit message: swap stupid trrs for usb-c
Parts:
- removed J1, J6: MJ-4PP-9, kbd:MJ-4PP-9, symbol Connector_Audio:AudioJack4
- added J5, J9: USB_C_Receptacle_USB2.0_16P, Connector_USB:USB_C_Receptacle_XKB_U262-16XN-4BVC11, symbol Connector:USB_C_Receptacle_USB2.0_16P
- RSW1, RSW2: footprint kbd:ResetSW -> Button_Switch_THT:SW_PUSH_1P1T_6x3.5mm_H4.3_APEM_MJTP1243; now fitted
- SW21, SW42: footprint kbd:keyswitch_cherrymx_alps_choc12_1.5u -> PCM_Switch_Keyboard_Cherry_MX:SW_Cherry_MX_PCB_1.00u
Connections:
- net GND: now also J9.A1 (GND), J9.A12 (GND), J9.B1 (GND), J9.B12 (GND), J9.S1 (SHIELD)
- net GNDA: now also J5.A1 (GND), J5.A12 (GND), J5.B1 (GND), J5.B12 (GND), J5.S1 (SHIELD)
- net bat+: now also J3.1 (Pin_1); no longer J3.2 (Pin_2)
- net bat+_r: now also J4.1 (Pin_1); no longer J4.2 (Pin_2)
- net bat-: now also J3.2 (Pin_2); no longer J3.1 (Pin_1)
- net bat-_r: now also J4.2 (Pin_2); no longer J4.1 (Pin_1)
- net data: now also J9.A6 (D+), J9.B6 (D+)
- net data_r: now also J5.A6 (D+), J5.B6 (D+)
- new net: J9.A4 (VBUS), J9.A9 (VBUS), J9.B4 (VBUS), J9.B9 (VBUS)
- new net: J5.A4 (VBUS), J5.A9 (VBUS), J5.B4 (VBUS), J5.B9 (VBUS)
- no-connect marks 26 -> 38
Other:
- note added: "changes from original corne v2.0 light 1. support for nice! nano (or nrf super micro) controllers 2. battery + on/off switch 3. usb-c for between half connection (not needed for wireless) 4. fix schematic/pcb such that drc/erc pass and are valid for kicad 8.0 (use default symbols where possible)"
- note removed: "TRS jack (backwards compatibility from non-wireless version)"
- company: foostan -> kevontheweb
- title: Corne Light -> Corne Light (wireless mod)
- moved on the sheet: D1, D10, D11, D12, D13, D14, D15, D16, D17, D18, D19, D2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

Commit message: put jacks back, erc and drc. finishing touches
Parts:
- removed J5, J9: USB_C_Receptacle_USB2.0_16P, Connector_USB:USB_C_Receptacle_XKB_U262-16XN-4BVC11, symbol Connector:USB_C_Receptacle_USB2.0_16P
- removed SW44, SW45: SW_Slide_DPDT, Button_Switch_THT:SW_CK_JS202011AQN_DPDT_Angled, symbol Switch:SW_Slide_DPDT
- added J6, J8: AudioJack4, custom:PJ320A, symbol Connector_Audio:AudioJack4
- added SW44, SW46: SW_SPDT, custom:MSK-12C01-07(1P2T), symbol Switch:SW_SPDT
Connections:
- net GND: now also J6.R1
- net GNDA: now also J8.R1
- net VCC: now also J6.R2
- net VDD: now also J8.R2
- net bat+: now also SW46.3 (C)
- net bat+_r: now also SW44.3 (C)
- net data: now also J6.T
- net data_r: now also J8.T
- net at U1.13 (BAT+), U1.29 (BAT+): now also SW46.2 (B)
- net at U2.13 (BAT+), U2.29 (BAT+): now also SW44.2 (B)
- no-connect marks 38 -> 20
